File: evc_seriously.sch (KiCad schematic (older format))
At the start: 58 parts, among them J1 Screw_Terminal_01x10, J2 Conn_ARM_JTAG_SWD_10, J3 J_IN, J4 J_OUT, SW1 SW_Push, U1 TCA9517, U2 MPM3510A, U3 MPM3510A, U4 STM32F303K8Tx, U5 MIC2981, U6 LM9022

Commit message: Start routing nets
- Routed GND, +5V, and some +3V3
- TODO: swap positions of 3V3 and 5V bucks to simplify power bus
Parts:
- C1, C2: PartNumber (none) -> CL21A475KBQNNNE
- J3, J4: symbol Connector_Generic:Conn_02x05_Counter_Clockwise -> Connector_Generic:Conn_02x05_Odd_Even
Connections:
- net +24V: now also J3.1 (Pin_1), J3.3 (Pin_3), J4.2 (Pin_2), J4.4 (Pin_4); no longer J3.10 (Pin_10), J3.9 (Pin_9), J4.10 (Pin_10), J4.9 (Pin_9)
- net +3V3: now also J3.9 (Pin_9); no longer J3.6 (Pin_6)
- net +3V3_B: now also J4.10 (Pin_10); no longer J4.6 (Pin_6)
- net GND: now also H1.1, H2.1, H3.1, H4.1, J3.10 (Pin_10), J3.6 (Pin_6), J3.8 (Pin_8), J4.7 (Pin_7), J4.9 (Pin_9); no longer J3.1 (Pin_1), J3.3 (Pin_3), J3.5 (Pin_5), J4.2 (Pin_2), J4.4 (Pin_4)
- net SCL_B: now also J4.8 (Pin_8); no longer J4.7 (Pin_7)
- net SDA_A: now also J3.5 (Pin_5); no longer J3.8 (Pin_8)
- net SDA_B: now also J4.6 (Pin_6); no longer J4.8 (Pin_8)
- net USR_SW: now also U4.25 (PA15); no longer U4.20 (PA10)
- no-connect marks 18 -> 14
Changed lines of the file:
@@
 $EndComp
 $Comp
-L Connector_Generic:Conn_02x05_Counter_Clockwise J4
+L Connector_Generic:Conn_02x05_Odd_Even J4
 U 1 1 5F7B231A
 P 9750 3450
@@
 $EndComp
 $Comp
-L Connector_Generic:Conn_02x05_Counter_Clockwise J3
+L Connector_Generic:Conn_02x05_Odd_Even J3
 U 1 1 5F7B26B3
-P 9750 2750
-F 0 "J3" H 9800 3050 50  0000 C CNN
-F 1 "J_IN" H 9800 2450 50  0000 C CNN
-F 2 "Connector_PinHeader_2.54mm:PinHeader_2x05_P2.54mm_Vertical" H 9750 2750 50  0001 C CNN
-F 3 "~" H 9750 2750 50  0001 C CNN
-	1    9750 2750
-	1    0    0    -1
+P 9850 2750
+F 0 "J3" H 9900 3050 50  0000 C CNN
+F 1 "J_IN" H 9900 2450 50  0000 C CNN
+F 2 "Connector_PinHeader_2.54mm:PinHeader_2x05_P2.54mm_Vertical" H 9850 2750 50  0001 C CNN
+F 3 "~" H 9850 2750 50  0001 C CNN
+	1    9850 2750
+	-1   0    0    1
 $EndComp
 Text Notes 7050 6975 0    50   ~ 0
@@
 Text Label 10400 2750 2    50   ~ 0
 SDA_A
-Text Label 10400 2850 2    50   ~ 0
+Text Label 10400 2650 2    50   ~ 0
 SCL_A
 $Comp
@@
 	9500 2950 9500 2850
 Wire Wire Line
-	10100 2650 10050 2650
-Wire Wire Line
-	10100 2550 10050 2550
-Wire Wire Line
-	10100 2550 10100 2650
+	10100 2950 10050 2950
+Wire Wire Line
+	10100 2850 10050 2850
+Wire Wire Line
+	10100 2850 10100 2950
 Wire Wire Line
 	9500 2850 9500 2750
@@
 	9500 2550 9550 2550
 Connection ~ 9500 2650
-Connection ~ 10100 2550
+Connection ~ 10100 2850
 Wire Wire Line
 	9400 2950 9500 2950
@@
 	10250 5350 10600 5350
 Wire Wire Line
-	10500 2550 10100 2550
+	10500 2850 10100 2850
 $Comp
 L power:+3.3V #PWR046
 U 1 1 5F8AECA8
-P 10500 2950
-F 0 "#PWR046" H 10500 2800 50  0001 C CNN
-F 1 "+3.3V" H 10515 3123 50  0000 C CNN
-F 2 "" H 10500 2950 50  0001 C CNN
-F 3 "" H 10500 2950 50  0001 C CNN
-	1    10500 2950
-	0    1    1    0
-$EndComp
-$Comp
-L power:+24V #PWR045
-U 1 1 5F8A71D3
 P 10500 2550
-F 0 "#PWR045" H 10500 2400 50  0001 C CNN
-F 1 "+24V" H 10515 2723 50  0000 C CNN
+F 0 "#PWR046" H 10500 2400 50  0001 C CNN
+F 1 "+3.3V" H 10515 2723 50  0000 C CNN
 F 2 "" H 10500 2550 50  0001 C CNN
 F 3 "" H 10500 2550 50  0001 C CNN
@@
 	0    1    1    0
 $EndComp
-Wire Wire Line
-	10500 2950 10050 2950
-Wire Wire Line
-	10400 2850 10050 2850
+$Comp
+L power:+24V #PWR045
+U 1 1 5F8A71D3
+P 10500 2850
+F 0 "#PWR045" H 10500 2700 50  0001 C CNN
+F 1 "+24V" H 10515 3023 50  0000 C CNN
+F 2 "" H 10500 2850 50  0001 C CNN
+F 3 "" H 10500 2850 50  0001 C CNN
+	1    10500 2850
+	0    1    1    0
+$EndComp
+Wire Wire Line
+	10500 2550 10050 2550
+Wire Wire Line
+	10400 2650 10050 2650
 Wire Wire Line
 	10400 2750 10050 2750
@@
 F 2 "Capacitor_SMD:C_0805_2012Metric" H 5788 1500 50  0001 C CNN
 F 3 "~" H 5750 1650 50  0001 C CNN
+F 4 "CL21A475KBQNNNE" H 5750 1650 50  0001 C CNN "PartNumber"
 	1    5750 1650
 	-1   0    0    1
@@
 F 2 "Capacitor_SMD:C_0805_2012Metric" H 5988 1500 50  0001 C CNN
 F 3 "~" H 5950 1650 50  0001 C CNN
+F 4 "CL21A475KBQNNNE" H 5950 1650 50  0001 C CNN "PartNumber"
 	1    5950 1650
 	-1   0    0    1
@@
 Text Notes 7050 6775 0    50   ~ 0
 MPS3510A monolithic buck regulator
-Wire Wire Line
-	5650 2550 5650 2650
 $Comp
 L power:+3.3V #PWR024
@@
 	1    0    0    -1
 $EndComp
-NoConn ~ 6250 4400
 NoConn ~ 6250 4100
 NoConn ~ 6250 3700
-NoConn ~ 5150 3900
 NoConn ~ 5150 3800
 NoConn ~ 5150 3500
@@
 Wire Wire Line
 	6250 4000 6600 4000
-Text Label 6600 3900 2    50   ~ 0
-USR_SW
-Wire Wire Line
-	6250 3900 6600 3900
 Text Label 4800 4000 0    50   ~ 0
 SWO
@@
 SWDCLK
 $Comp
+L Mechanical:MountingHole_Pad H2
+U 1 1 5F89B3C6
+P 1250 1150
+F 0 "H2" H 1350 1199 50  0000 L CNN
+F 1 "MountingHole_Pad" H 1350 1108 50  0000 L CNN
+F 2 "MountingHole:MountingHole_3.2mm_M3_Pad" H 1250 1150 50  0001 C CNN
+F 3 "~" H 1250 1150 50  0001 C CNN
+	1    1250 1150
+	1    0    0    -1
+$EndComp
+$Comp
+L Mechanical:MountingHole_Pad H3
+U 1 1 5F89B9F1
+P 1450 1150
+F 0 "H3" H 1550 1199 50  0000 L CNN
+F 1 "MountingHole_Pad" H 1550 1108 50  0000 L CNN
+F 2 "MountingHole:MountingHole_3.2mm_M3_Pad" H 1450 1150 50  0001 C CNN
+F 3 "~" H 1450 1150 50  0001 C CNN
+	1    1450 1150
+	1    0    0    -1
+$EndComp
+$Comp
+L Mechanical:MountingHole_Pad H4
+U 1 1 5F89BFB4
+P 1650 1150
+F 0 "H4" H 1750 1199 50  0000 L CNN
+F 1 "MountingHole_Pad" H 1750 1108 50  0000 L CNN
+F 2 "MountingHole:MountingHole_3.2mm_M3_Pad" H 1650 1150 50  0001 C CNN
+F 3 "~" H 1650 1150 50  0001 C CNN
+	1    1650 1150
+	1    0    0    -1
+$EndComp
+$Comp
+L Mechanical:MountingHole_Pad H1
+U 1 1 5F896868
+P 1050 1150
+F 0 "H1" H 1150 1199 50  0000 L CNN
+F 1 "MountingHole_Pad" H 1150 1108 50  0000 L CNN
+F 2 "MountingHole:MountingHole_3.2mm_M3_Pad" H 1050 1150 50  0001 C CNN
+F 3 "~" H 1050 1150 50  0001 C CNN
+	1    1050 1150
+	1    0    0    -1
+$EndComp
+$Comp
+L power:GND #PWR0102
+U 1 1 5F8E4081
+P 1650 1350
+F 0 "#PWR0102" H 1650 1100 50  0001 C CNN
+F 1 "GND" H 1655 1177 50  0000 C CNN
+F 2 "" H 1650 1350 50  0001 C CNN
+F 3 "" H 1650 1350 50  0001 C CNN
+	1    1650 1350
+	1    0    0    -1
+$EndComp
+Wire Wire Line
+	1650 1350 1650 1300
+Wire Wire Line
+	1650 1300 1450 1300
+Wire Wire Line
+	1450 1300 1450 1250
+Connection ~ 1650 1300
+Wire Wire Line
+	1650 1300 1650 1250
+Wire Wire Line
+	1450 1300 1250 1300
+Wire Wire Line
+	1250 1300 1250 1250
+Connection ~ 1450 1300
+Wire Wire Line
+	1250 1300 1050 1300
+Wire Wire Line
+	1050 1300 1050 1250
+Connection ~ 1250 1300
+NoConn ~ 5150 3900
+Text Label 6600 4400 2    50   ~ 0
+USR_SW
+Wire Wire Line
+	5650 2550 5650 2650
+$Comp
 L MCU_ST_STM32F3:STM32F303K8Tx U4
 U 1 1 5F7AE5D9
@@
 	1    0    0    -1
 $EndComp
-$Comp
-L Mechanical:MountingHole_Pad H2
-U 1 1 5F89B3C6
-P 1250 1150
-F 0 "H2" H 1350 1199 50  0000 L CNN
-F 1 "MountingHole_Pad" H 1350 1108 50  0000 L CNN
-F 2 "MountingHole:MountingHole_3.2mm_M3_Pad" H 1250 1150 50  0001 C CNN
-F 3 "~" H 1250 1150 50  0001 C CNN
-	1    1250 1150
-	1    0    0    -1
-$EndComp
-$Comp
-L Mechanical:MountingHole_Pad H3
-U 1 1 5F89B9F1
-P 1450 1150
-F 0 "H3" H 1550 1199 50  0000 L CNN
-F 1 "MountingHole_Pad" H 1550 1108 50  0000 L CNN
-F 2 "MountingHole:MountingHole_3.2mm_M3_Pad" H 1450 1150 50  0001 C CNN
-F 3 "~" H 1450 1150 50  0001 C CNN
-	1    1450 1150
-	1    0    0    -1
-$EndComp
-$Comp
-L Mechanical:MountingHole_Pad H4
-U 1 1 5F89BFB4
-P 1650 1150
-F 0 "H4" H 1750 1199 50  0000 L CNN
-F 1 "MountingHole_Pad" H 1750 1108 50  0000 L CNN
-F 2 "MountingHole:MountingHole_3.2mm_M3_Pad" H 1650 1150 50  0001 C CNN
-F 3 "~" H 1650 1150 50  0001 C CNN
-	1    1650 1150
-	1    0    0    -1
-$EndComp
-$Comp
-L Mechanical:MountingHole_Pad H1
-U 1 1 5F896868
-P 1050 1150
-F 0 "H1" H 1150 1199 50  0000 L CNN
-F 1 "MountingHole_Pad" H 1150 1108 50  0000 L CNN
-F 2 "MountingHole:MountingHole_3.2mm_M3_Pad" H 1050 1150 50  0001 C CNN
-F 3 "~" H 1050 1150 50  0001 C CNN
-	1    1050 1150
-	1    0    0    -1
-$EndComp
-NoConn ~ 1050 1250
-NoConn ~ 1250 1250
-NoConn ~ 1450 1250
-NoConn ~ 1650 1250
+NoConn ~ 6250 3900
+Wire Wire Line
+	6600 4400 6250 4400
 $EndSCHEMATC
